File: LoRa-BikeLink-TX/LoRa-BikeLink-TX.kicad_pcb (KiCad board)
At the start: 2 copper layers, 95 x 20 mm, 10 parts, among them P1 CONN_01X02, P2 CONN_01X04, P3 CONN_01X02, U1 RFM95, U2 ADXL345_brkout

Commit message: Some text
Parts:
- C1: footprint Capacitors_SMD:C_1206_HandSoldering -> Capacitors_SMD:C_1206
- R1: value 100k -> 39k; footprint Resistors_SMD:R_1206_HandSoldering -> Resistors_SMD:R_0805_HandSoldering
- R2: value 100k -> 120k; footprint Resistors_SMD:R_1206_HandSoldering -> Resistors_SMD:R_0805_HandSoldering
- R3: footprint Resistors_SMD:R_1206_HandSoldering -> Resistors_SMD:R_0805_HandSoldering
- uP1: footprint ArduProMini_only_sideholes -> MyLib:ArduProMini_only_sideholes
- moved R3 5.39 mm to (134.0, 110.0)
- moved R1 4.53 mm to (123.5, 106.5)
- moved P2 4.47 mm to (95.0, 117.0)
- moved U2 3.50 mm to (90.5, 107.0)
- moved P1 2.55 mm to (169.5, 109.5)
- moved P3 2.06 mm to (77.0, 109.5), turned to 90 degrees
- moved R2 1.80 mm to (123.5, 109.0), turned to 180 degrees
- moved C1 0.50 mm to (166.0, 114.5), turned to 0 degrees
Connections:
- P2 pad 4: (no net) -> /BATT_IN

Commit message: PDF
Parts:
- removed R3: 100k, Resistors_SMD:R_0805_HandSoldering
- C1: value 10u -> 0.1u
- moved P2 5.70 mm to (100.5, 118.5)
- moved U2 5.00 mm to (95.5, 107.0)
- moved P1 4.50 mm to (174.0, 109.5)
- moved P3 3.64 mm to (80.5, 110.5)
- moved U1 3.00 mm to (154.0, 110.0)
- moved uP1 3.00 mm to (124.0, 110.0)
- moved C1 1.80 mm to (167.5, 113.5), turned to 270 degrees
Connections:
- net /RF_DIO1 renamed /Lora_DIO1
- P2 pad 4: /BATT_IN -> (no net)
- U1 pad 14: /RF_INT_OUT -> /Lora_DIO0
- U1 pad 5: Net-(R3-Pad2) -> Net-(U1-Pad5)
- U1 pad 6: (no net) -> /Lora_RESET
- U2 pad 1: (no net) -> /PWR_OUT
- U2 pad 10: /PWR_OUT -> (no net)
- uP1 pad 11: /ACC_INT1 -> /Lora_DIO0
- uP1 pad 12: /RF_INT_OUT -> /ACC_INT1
- uP1 pad 18: (no net) -> /Lora_RESET
- uP1 pad 20: (no net) -> GND
- uP1 pad 30: (no net) -> Net-(U1-Pad5)
Routing:
- net /PWR_OUT: track 0.00 -> 58.1 mm, vias 0 -> 2
- net /Lora_DIO0: track 0.00 -> 46.7 mm, vias 0 -> 2
- net /Lora_DIO1: track 0.00 -> 39.6 mm, vias 0 -> 2
- net /Lora_RESET: track 0.00 -> 26.5 mm
- net /Lora_SCK: track 0.00 -> 22.9 mm, vias 0 -> 2
- net /Lora_MISO: track 0.00 -> 20.0 mm
- net /Lora_MOSI: track 0.00 -> 17.0 mm
- net Net-(P1-Pad1): track 0.00 -> 14.5 mm
- net Net-(U1-Pad5): track 0.00 -> 12.8 mm
- net /ADC_0: track 0.00 -> 8.14 mm
Other:
- board size 95 x 20 mm -> 100 x 20 mm

Commit message: Update
Parts:
- P2: footprint MyLib:TPS61200_Tiny_Module -> TPS61200_Tiny_Module
- P3: moved to B.Cu
- U2: footprint MyLib:ADXL345_BRKOUT -> ADXL345_BRKOUT
- uP1: footprint MyLib:ArduProMini_only_sideholes -> ArduProMini_only_sideholes
- moved P2 20.2 mm to (90.5, 101.0), turned to 270 degrees
- moved U2 3.00 mm to (95.5, 110.0)
- moved P3 2.50 mm to (83.0, 110.5), turned to 270 degrees
- moved P1 0.16 mm to (173.8, 109.5)
Routing:
- net /BATT_IN: track 0.00 -> 45.3 mm, vias 0 -> 1
- net /ACC_INT1: track 0.00 -> 43.7 mm
- net /PWR_OUT: track 58.1 -> 94.2 mm, vias 2 -> 4

Commit message: Update
Parts:
- removed P3: CONN_01X02, Connectors:PINHEAD1-2
- added J1: CONN_01X01, Wire_Pads:SolderWirePad_single_SMD_5x10mm, F.Cu at (79.5, 110.0)
- added J2: CONN_01X01, Wire_Pads:SolderWirePad_single_SMD_5x10mm, F.Cu at (79.5, 116.5)
- added J3: CONN_01X01, Wire_Pads:SolderWirePad_single_SMD_5x10mm, B.Cu at (79.5, 110.0)
- P2: footprint TPS61200_Tiny_Module -> MyLib:TPS61200_Tiny_Module
- U2: footprint ADXL345_BRKOUT -> MyLib:ADXL345_BRKOUT
- uP1: footprint ArduProMini_only_sideholes -> MyLib:ArduProMini_only_sideholes
Routing:
- net /BATT_IN: track 45.3 -> 66.5 mm, vias 1 -> 2
Other:
- board size 100 x 20 mm -> 100 x 19 mm
- net class Batt added: clearance 0.5, trace_width 1, via_dia 0.8, via_drill 0.6
