File: BikeLink-TX-PCB/LoRa-BikeLink-TX.kicad_pcb (KiCad board)
At the start: 2 copper layers, 100 x 19 mm, 11 parts, among them J1 CONN_01X01, J2 CONN_01X01, J3 CONN_01X01, P1 CONN_01X02, P2 CONN_01X04, U1 RFM95, U2 ADXL345_brkout

Commit message: 1st code
Routing:
- net /PWR_OUT: track 93.8 -> 95.1 mm
Other:
- net class Batt: clearance 0.5 -> 0.6
Changed lines of the file:
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@@
     (thickness 1.6)
     (drawings 4)
-    (tracks 82)
+    (tracks 88)
     (zones 0)
     (modules 11)
@@
     (mod_text_size 1 1)
     (mod_text_width 0.15)
-    (pad_size 1.524 1.524)
-    (pad_drill 0.762)
+    (pad_size 1.8 1.8)
+    (pad_drill 1)
     (pad_to_mask_clearance 0.2)
     (aux_axis_origin 101.5 112)
@@
   )
   (net_class Batt ""
-    (clearance 0.5)
+    (clearance 0.6)
     (trace_width 1)
     (via_dia 1)
@@
   (segment (start 163.25 100.25) (end 163.25 94.72) (width 0.5) (layer B.Cu) (net 3))
   (segment (start 168.5 105.5) (end 163.25 100.25) (width 0.5) (layer B.Cu) (net 3))
-  (segment (start 158.17 94.72) (end 158.17 103.17) (width 0.5) (layer B.Cu) (net 4))
-  (segment (start 168.5 103.5) (end 172.5 103.5) (width 0.5) (layer B.Cu) (net 4))
-  (via (at 168.5 103.5) (size 1) (drill 0.6) (layers F.Cu B.Cu) (net 4))
-  (segment (start 158.5 103.5) (end 168.5 103.5) (width 0.5) (layer F.Cu) (net 4))
-  (via (at 158.5 103.5) (size 1) (drill 0.6) (layers F.Cu B.Cu) (net 4))
-  (segment (start 158.17 103.17) (end 158.5 103.5) (width 0.5) (layer B.Cu) (net 4))
+  (segment (start 172.9 103.5) (end 169 103.5) (width 0.5) (layer B.Cu) (net 4))
+  (segment (start 169 103.5) (end 168.5 103) (width 0.5) (layer B.Cu) (net 4))
+  (segment (start 158.17 94.72) (end 158.17 102.67) (width 0.5) (layer B.Cu) (net 4))
+  (segment (start 158.17 102.67) (end 158.5 103) (width 0.5) (layer B.Cu) (net 4))
+  (via (at 168.5 103) (size 1) (drill 0.6) (layers F.Cu B.Cu) (net 4))
+  (segment (start 158.5 103) (end 168.5 103) (width 0.5) (layer F.Cu) (net 4))
+  (via (at 158.5 103) (size 1) (drill 0.6) (layers F.Cu B.Cu) (net 4))
   (segment (start 190.5 95.5) (end 194 95.5) (width 0.5) (layer B.Cu) (net 5))
   (segment (start 196 102) (end 199.6585 102) (width 0.5) (layer B.Cu) (net 5))
@@
   (segment (start 195 96.5) (end 195 101) (width 0.5) (layer B.Cu) (net 5))
   (segment (start 194 95.5) (end 195 96.5) (width 0.5) (layer B.Cu) (net 5))
+  (segment (start 119.75 97.5) (end 119.27 97.02) (width 1) (layer F.Cu) (net 6))
+  (segment (start 119.27 97.02) (end 119.27 94.77) (width 1) (layer F.Cu) (net 6))
+  (segment (start 119.75 98.5) (end 119.75 97.5) (width 1) (layer F.Cu) (net 6))
+  (segment (start 122 98.5) (end 119.75 98.5) (width 1) (layer B.Cu) (net 6))
   (via (at 115 95) (size 1) (drill 0.6) (layers F.Cu B.Cu) (net 6))
   (segment (start 195 104.5) (end 194 103.5) (width 1) (layer B.Cu) (net 6))
@@
   (segment (start 122 98.5) (end 144 98.5) (width 1) (layer B.Cu) (net 6))
   (segment (start 144 98.5) (end 145.5 97) (width 1) (layer B.Cu) (net 6))
-  (segment (start 119.27 94.77) (end 119.27 95.77) (width 1) (layer F.Cu) (net 6))
-  (segment (start 119.27 95.77) (end 122 98.5) (width 1) (layer F.Cu) (net 6))
-  (via (at 122 98.5) (size 1) (drill 0.6) (layers F.Cu B.Cu) (net 6))
+  (via (at 119.75 98.5) (size 1) (drill 0.6) (layers F.Cu B.Cu) (net 6))
   (segment (start 119.27 94.77) (end 115.23 94.77) (width 0.5) (layer F.Cu) (net 6))
   (segment (start 115 95) (end 115 98.5) (width 0.5) (layer B.Cu) (net 6))
@@
   (segment (start 185.5 107.5) (end 153.5 107.5) (width 0.5) (layer F.Cu) (net 14))
   (via (at 185.5 107.5) (size 1) (drill 0.6) (layers F.Cu B.Cu) (net 14))
-  (segment (start 190.5 105.5) (end 185.5 105.5) (width 0.5) (layer B.Cu) (net 15))
+  (segment (start 190.1 105.5) (end 185.7034 105.5) (width 0.5) (layer B.Cu) (net 15))
+  (segment (start 185.7034 105.5) (end 185.4978 105.2944) (width 0.5) (layer B.Cu) (net 15))
+  (segment (start 148.01 105.99) (end 148.000001 105.980001) (width 0.5) (layer B.Cu) (net 15))
+  (segment (start 148.000001 105.980001) (end 148.000001 105.799999) (width 0.5) (layer B.Cu) (net 15))
+  (segment (start 148.000001 105.799999) (end 148.5 105.3) (width 0.5) (layer B.Cu) (net 15))
   (segment (start 148.01 105.99) (end 148.01 109.96) (width 0.5) (layer B.Cu) (net 15))
-  (segment (start 148.5 105.5) (end 148.01 105.99) (width 0.5) (layer B.Cu) (net 15))
-  (via (at 148.5 105.5) (size 1) (drill 0.6) (layers F.Cu B.Cu) (net 15))
-  (segment (start 185.5 105.5) (end 148.5 105.5) (width 0.5) (layer F.Cu) (net 15))
-  (via (at 185.5 105.5) (size 1) (drill 0.6) (layers F.Cu B.Cu) (net 15))
+  (via (at 148.5 105.3) (size 1) (drill 0.6) (layers F.Cu B.Cu) (net 15))
+  (segment (start 185.5 105.3) (end 148.5 105.3) (width 0.5) (layer F.Cu) (net 15))
+  (via (at 185.4978 105.2944) (size 1) (drill 0.6) (layers F.Cu B.Cu) (net 15))
   (zone (net 1) (net_name GND) (layer F.Cu) (hatch edge 0.508)
     (connect_pads (clearance 0.508))
@@
       )
     )
+  )
+  (zone (net 0) (net_name "") (layer B.Cu) (hatch edge 0.508)
+    (connect_pads (clearance 0.508))
+    (min_thickness 0.254)
+    (keepout (tracks not_allowed) (vias not_allowed) (copperpour not_allowed))
+    (fill yes (arc_segments 16) (thermal_gap 0.508) (thermal_bridge_width 0.508))
+    (polygon
+      (pts
+        (xy 193.75 105.25) (xy 193.75 106.75) (xy 196.25 106.75) (xy 196.25 105.25)
+      )
+    )
+  )
+  (zone (net 0) (net_name "") (layer B.Cu) (hatch edge 0.508)
+    (connect_pads (clearance 0.508))
+    (min_thickness 0.254)
+    (keepout (tracks allowed) (vias allowed) (copperpour not_allowed))
+    (fill yes (arc_segments 16) (thermal_gap 0.508) (thermal_bridge_width 0.508))
+    (polygon
+      (pts
+        (xy 175 108.75) (xy 175 96.25) (xy 175.75 96.25) (xy 175.75 108.75)
+      )
+    )
+  )
+  (zone (net 0) (net_name "") (layer B.Cu) (hatch edge 0.508)
+    (connect_pads (clearance 0.508))
+    (min_thickness 0.254)
+    (keepout (tracks allowed) (vias allowed) (copperpour not_allowed))
+    (fill yes (arc_segments 16) (thermal_gap 0.508) (thermal_bridge_width 0.508))
+    (polygon
+      (pts
+        (xy 188 98.25) (xy 188 110.25) (xy 187 110.25) (xy 187 98.25)
+      )
+    )
+  )
+  (zone (net 0) (net_name "") (layer B.Cu) (hatch edge 0.508)
+    (connect_pads (clearance 0.508))
+    (min_thickness 0.254)
+    (keepout (tracks allowed) (vias allowed) (copperpour not_allowed))
+    (fill yes (arc_segments 16) (thermal_gap 0.508) (thermal_bridge_width 0.508))
+    (polygon
+      (pts
+        (xy 188 96.75) (xy 188 94.5) (xy 187 94.5) (xy 187 96.75)
+      )
+    )
